File: PCBs/Rocket_01/Rocket_01.kicad_sch (KiCad schematic)
At the start: 14 parts, among them Q1 NTR3C21NZ, U1 MSP430G2210ID, U2 TPS61220DCK

Commit message: update of the schematic Rocket_01
first complete version
Parts:
- added BT1: Battery_Cell, symbol Device:Battery_Cell
- added D3, D4, D5: LED_Filled, LED_SMD:LED_0805_2012Metric_Pad1.15x1.40mm_HandSolder, symbol Device:LED_Filled
- added D6: SS2040LL, Diode_SMD:D_SOD-123F, symbol Device:D_Schottky
- added GND, Trigger: ~, symbol Connector:TestPoint
- added L4: 1mH, Inductor_SMD:L_APV_ANR8040, symbol Device:L
- added Q2: NTR3C21NZ, symbol Transistor_FET:Q_NMOS_GSD
- L2: value 4.7uH -> 1mH; footprint Inductor_SMD:L_Changjiang_FNR3015S -> Inductor_SMD:L_APV_ANR8040
- R1: value R -> 9.1kR
- R2: value R -> 1.0kR
Connections:
- net +5V: now also D6.1 (K), L4.1
- net GND: now also BT1.2 (-), GND.1, Q2.2 (S)
- net at D1.2 (A): now also D3.1 (K); no longer L2.2
- net at U1.4 (TA0.1/CA2/P1.2): now also Trigger.1
- net at U1.7 (TA0.0/CA5/P1.5): now also Q2.1 (G)
- net +3.3V renamed +3.0V
- net +3.0V: now also BT1.1 (+)
- new net: D3.2 (A), L4.2
- new net: D4.1 (K), D5.2 (A)
- new net: D4.2 (A), L2.2
- new net: D5.1 (K), D6.2 (A), Q2.3 (D)
Other:
- note added: "1.8V up to 3.6V"
- note added: "500mV"
- note added: "Fmax = approx. 100kHz"
- note added: "up to 5.5V, up to 100mA"
